File: Rain connectors/_autosave-Rain connectors.kicad_sch (KiCad schematic)
At the start: 7 parts, among them J1 Conn_01x06_Socket, J2 Conn_01x06_Socket, J3 Conn_01x03_Socket

Commit message: Check to see if the rain connectors v.2. needs updating
Parts:
- J1, J2: footprint Connector_JST:JST_PH_S6B-PH-SM4-TB_1x06-1MP_P2.00mm_Horizontal -> Connector_JST:JST_XA_S06B-XASK-1N-BN_1x06_P2.50mm_Horizontal
- J3: footprint Connector_PinHeader_2.00mm:PinHeader_1x03_P2.00mm_Horizontal -> Connector_PinHeader_2.00mm:PinHeader_1x03_P2.00mm_Vertical
Connections:
- net +5V: now also J3.1 (Pin_1)
- net GND: no longer J3.1 (Pin_1)
Changed lines of the file:
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@@
-	)
-	(junction
-		(at 160.02 105.41)
-		(diameter 0)
-		(color 0 0 0 0)
 	)
 	(junction
@@
 	(wire
 		(pts
-			(xy 124.46 105.41) (xy 160.02 105.41)
-		)
-		(stroke
-			(width 0)
-			(type default)
-		)
-	)
-	(wire
-		(pts
-			(xy 160.02 105.41) (xy 161.29 105.41)
+			(xy 124.46 105.41) (xy 161.29 105.41)
 		)
 		(stroke
@@
 	(wire
 		(pts
-			(xy 144.78 127) (xy 160.02 127)
+			(xy 144.78 127) (xy 158.75 127)
 		)
 		(stroke
@@
 	(wire
 		(pts
+			(xy 158.75 92.71) (xy 158.75 127)
+		)
+		(stroke
+			(width 0)
+			(type default)
+		)
+	)
+	(wire
+		(pts
 			(xy 146.05 119.38) (xy 146.05 123.19)
 		)
@@
 		(pts
 			(xy 138.43 119.38) (xy 138.43 123.19)
-		)
-		(stroke
-			(width 0)
-			(type default)
-		)
-	)
-	(wire
-		(pts
-			(xy 160.02 127) (xy 160.02 105.41)
 		)
 		(stroke
@@
 			)
 		)
-		(property "Footprint" "Connector_JST:JST_PH_S6B-PH-SM4-TB_1x06-1MP_P2.00mm_Horizontal"
+		(property "Footprint" "Connector_JST:JST_XA_S06B-XASK-1N-BN_1x06_P2.50mm_Horizontal"
 			(at 166.37 97.79 0)
 			(effects
@@
 			)
 		)
-		(property "Footprint" "Connector_JST:JST_PH_S6B-PH-SM4-TB_1x06-1MP_P2.00mm_Horizontal"
+		(property "Footprint" "Connector_JST:JST_XA_S06B-XASK-1N-BN_1x06_P2.50mm_Horizontal"
 			(at 111.76 100.33 0)
 			(effects
@@
 			)
 		)
-		(property "Footprint" "Connector_PinHeader_2.00mm:PinHeader_1x03_P2.00mm_Horizontal"
+		(property "Footprint" "Connector_PinHeader_2.00mm:PinHeader_1x03_P2.00mm_Vertical"
 			(at 142.24 132.08 0)
 			(effects
