File: Light Control Board/LightControlBoard.kicad_pcb (KiCad board)
At the start: 2 copper layers, 50.7 x 101.1 mm, 25 parts, among them J1 8P8C, J2 8P8C, J3 RJ45, J4 RJ45, J5 Screw_Terminal_01x02, U6 OKI-78SR

Commit message: Rev. 3
Connections:
- U1 pad 31: Net-(U2-STB) -> Net-(U2-NC,Vio)
- U2 pad 5: GND -> Net-(U2-NC,Vio)
- U2 pad 8: Net-(U2-STB) -> GND
Routing:
- net Net-(U2-NC,Vio): track 0.00 -> 21.6 mm, vias 0 -> 1
- net Net-(U2-STB): track 17.5 -> 0.00 mm, vias 1 -> 0
- net GND: track 23.3 -> 21.2 mm, vias 3 -> 4
Other:
- board text added: "330_ Combined Sewer System LED Strip Controller Rev.3"
- board text removed: "330_ Combined Sewer System LED Strip Controller Rev.2"
