File: Light Control Board/LightControlBoard.kicad_sch (KiCad schematic)
At the start: 21 parts, among them J1 8P8C, J2 8P8C, J3 RJ45, J4 RJ45, J5 Screw_Terminal_01x02, U6 OKI-78SR

Commit message: Rev. 3
Connections:
- net GND: now also U2.8 (STB); no longer U2.5 (NC,Vio)
- net at U1.31 (3.3V): now also U2.5 (NC,Vio); no longer U2.8 (STB)
Changed lines of the file:
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@@
-	)
-	(junction
-		(at 224.79 118.11)
-		(diameter 0)
-		(color 0 0 0 0)
 	)
 	(junction
@@
 	(wire
 		(pts
-			(xy 232.41 111.76) (xy 232.41 118.11)
+			(xy 232.41 114.3) (xy 204.47 114.3)
 		)
 		(stroke
@@
 	(wire
 		(pts
+			(xy 232.41 111.76) (xy 232.41 114.3)
+		)
+		(stroke
+			(width 0)
+			(type default)
+		)
+	)
+	(wire
+		(pts
+			(xy 231.14 111.76) (xy 232.41 111.76)
+		)
+		(stroke
+			(width 0)
+			(type default)
+		)
+	)
+	(wire
+		(pts
 			(xy 215.9 109.22) (xy 218.44 109.22)
 		)
@@
 	(wire
 		(pts
-			(xy 231.14 101.6) (xy 199.39 101.6)
-		)
-		(stroke
-			(width 0)
-			(type default)
-		)
-	)
-	(wire
-		(pts
 			(xy 219.71 43.18) (xy 219.71 48.26)
 		)
@@
 	(wire
 		(pts
+			(xy 204.47 101.6) (xy 199.39 101.6)
+		)
+		(stroke
+			(width 0)
+			(type default)
+		)
+	)
+	(wire
+		(pts
 			(xy 80.01 71.12) (xy 85.09 71.12)
 		)
@@
 	(wire
 		(pts
-			(xy 231.14 111.76) (xy 232.41 111.76)
-		)
-		(stroke
-			(width 0)
-			(type default)
-		)
-	)
-	(wire
-		(pts
 			(xy 105.41 90.17) (xy 93.98 90.17)
 		)
@@
 	(wire
 		(pts
-			(xy 232.41 118.11) (xy 224.79 118.11)
-		)
-		(stroke
-			(width 0)
-			(type default)
-		)
-	)
-	(wire
-		(pts
 			(xy 100.33 68.58) (xy 100.33 49.53)
 		)
@@
 		(pts
 			(xy 39.37 45.72) (xy 40.64 45.72)
+		)
+		(stroke
+			(width 0)
+			(type default)
+		)
+	)
+	(wire
+		(pts
+			(xy 204.47 114.3) (xy 204.47 101.6)
 		)
 		(stroke
@@
 					(unit 1)
 				)
+			)
+		)
+	)
+	(symbol
+		(lib_id "power:GND")
+		(at 231.14 101.6 180)
+		(unit 1)
+		(exclude_from_sim no)
+		(in_bom yes)
+		(on_board yes)
+		(dnp no)
+		(fields_autoplaced yes)
+		(property "Reference" "#PWR02"
+			(at 231.14 95.25 0)
+			(effects
+				(font
+					(size 1.27 1.27)
+				)
+				(hide yes)
+			)
+		)
+		(property "Value" "GND"
+			(at 231.14 96.52 0)
+			(effects
+				(font
+					(size 1.27 1.27)
+				)
+			)
+		)
+		(property "Footprint" ""
+			(at 231.14 101.6 0)
+			(effects
+				(font
+					(size 1.27 1.27)
+				)
+				(hide yes)
+			)
+		)
+		(property "Datasheet" ""
+			(at 231.14 101.6 0)
+			(effects
+				(font
+					(size 1.27 1.27)
+				)
+				(hide yes)
+			)
+		)
+		(property "Description" "Power symbol creates a global label with name \"GND\" , ground"
+			(at 231.14 101.6 0)
+			(effects
+				(font
+					(size 1.27 1.27)
+				)
+				(hide yes)
+			)
+		)
+		(pin "1"
+		)
+		(instances
+			(project "LightControlBoard"
+				(path "/7f24777d-b764-439e-a42b-2ba1b91f0330"
+					(reference "#PWR02")
+					(unit 1)
+				)
