File: Rain and Switches Control Board/Rain and Switches Control Board.kicad_pcb (KiCad board)
At the start: 2 copper layers, 81.3 x 75.7 mm, 40 parts, among them J1 Conn_01x06_MountingPin, J2 Screw_Terminal_01x02, J3 Conn_01x02, J4 8P8C, J5 Conn_01x02, J6 Conn_01x02, J7 Conn_01x02, J8 Conn_01x02, J9 RJ45, Q1 NPN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

Commit message: Rev. 3
Parts:
- removed the REF** at (111.1, 43.4)
- removed the REF** at (111.1, 93.4)
- removed the REF** at (157.1, 43.4)
- removed the REF** at (166.1, 93.4)
- added J10: Conn_01x02, TerminalBlock:TerminalBlock_Altech_AK300-2_P5.00mm, F.Cu at (135.9, 88.5)
- added J11: Conn_01x02, TerminalBlock:TerminalBlock_Altech_AK300-2_P5.00mm, F.Cu at (135.9, 100.0)
- added REF**: MountingHole_3.2mm_M3, MountingHole:MountingHole_3.2mm_M3, F.Cu at (152.4, 95.0)
- added REF**: MountingHole_3.2mm_M3, MountingHole:MountingHole_3.2mm_M3, F.Cu at (184.9, 68.3)
- added REF**: MountingHole_3.2mm_M3, MountingHole:MountingHole_3.2mm_M3, F.Cu at (152.3, 50.5)
- moved U3 73.2 mm to (189.2, 53.0), turned to -90 degrees
- moved J1 69.7 mm to (137.6, 42.6), turned to -90 degrees
- moved J8 67.0 mm to (206.6, 99.7), turned to 0 degrees
- moved U2 59.7 mm to (186.1, 42.0)
- moved Q5 44.9 mm to (152.4, 60.3), turned to -90 degrees
- moved R11 44.7 mm to (158.0, 62.5), turned to -90 degrees
- moved J7 44.6 mm to (195.3, 99.7), turned to 0 degrees
- moved R16 42.2 mm to (148.2, 61.8)
- moved R10 37.6 mm to (158.0, 68.0), turned to -90 degrees
- moved Q4 37.2 mm to (152.4, 65.8), turned to -90 degrees
- moved R3 36.7 mm to (189.8, 84.2)
- moved R5 36.7 mm to (184.3, 84.2)
- moved U4 36.5 mm to (183.3, 81.4)
- moved R4 36.2 mm to (191.1, 73.4)
- moved R2 36.2 mm to (185.6, 73.4)
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Connections:
- U1 pad 26: unconnected-(U1-D19-Pad26) -> Net-(J11-Pin_2)
- U1 pad 27: unconnected-(U1-D20-Pad27) -> Net-(J10-Pin_2)
- U1 pad 31: Net-(U3-STB) -> Net-(U3-NC,Vio)
- U3 pad 1: Net-(U1-D23) -> Net-(U1-D22)
- U3 pad 4: Net-(U1-D22) -> Net-(U1-D23)
- U3 pad 5: GND -> Net-(U3-NC,Vio)
- U3 pad 8: Net-(U3-STB) -> GND
Routing:
- net Net-(J11-Pin_2): track 0.00 -> 72.4 mm
- net Net-(J10-Pin_2): track 0.00 -> 68.2 mm
- net Net-(J3-Pin_2): track 99.1 -> 43.5 mm
- net Net-(U3-CA_NH): track 78.6 -> 28.0 mm
- net Net-(U3-CA_NL): track 78.3 -> 28.2 mm
- net GND: track 80.8 -> 38.8 mm, vias 2 -> 4
- net Net-(J5-Pin_2): track 83.8 -> 43.1 mm
- net +12V: track 61.3 -> 23.9 mm
- net Net-(J6-Pin_2): track 66.9 -> 41.1 mm
- net /So5: track 4.86 -> 21.2 mm, vias 0 -> 1
- net Net-(U3-NC,Vio): track 0.00 -> 16.2 mm, vias 0 -> 1
- net Net-(U3-STB): track 16.0 -> 0.00 mm
- net Net-(J1-Pin_6): track 14.8 -> 29.5 mm
- net Net-(J7-Pin_2): track 59.0 -> 44.4 mm
- net /So4: track 4.23 -> 18.2 mm, vias 0 -> 1
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Other:
- board size 81.3 x 75.7 mm -> 86 x 69.3 mm
- board text added: "330 Combined Sewer System Rain Controller Rev. 3"
- board text added: "D10"
- board text added: "D14"
- board text added: "D15"
- board text added: "D16"
- board text added: "D17"
- board text added: "D18"
- board text added: "D19"
- board text added: "D20"
- board text added: "D6"
- board text added: "D7"
- board text added: "D8"
- board text added: "D9"
- board text removed: "330_Combined Sewer System Rain Controller Rev. 2"
- board text removed: "COM"
